Commit message: Implement PyBullet training pipeline and YOLO detector

File: training/robot_arm.urdf (robot description, URDF)
Before this commit: robot placeholder_robot_arm, 1 links, 0 joints
Links:
- added link end_effector, mass 0.05; collision sphere radius=0.02; visual sphere radius=0.02
- added link link1, mass 0.5; collision box size=0.05 0.05 0.1; visual box size=0.05 0.05 0.1
- added link link2, mass 0.4; collision box size=0.2 0.04 0.04; visual box size=0.2 0.04 0.04
- added link link3, mass 0.3; collision box size=0.2 0.04 0.04; visual box size=0.2 0.04 0.04
- added link link4, mass 0.25; collision box size=0.16 0.04 0.04; visual box size=0.16 0.04 0.04
- added link link5, mass 0.2; collision box size=0.12 0.04 0.04; visual box size=0.12 0.04 0.04
- added link link6, mass 0.15; collision box size=0.1 0.04 0.04; visual box size=0.1 0.04 0.04
- link base_link: mass None -> 1; geometry collision cylinder length=0.04 radius=0.06; visual cylinder length=0.04 radius=0.06
Joints:
- added joint ee_fixed: type fixed, parent link6, child end_effector, origin xyz=0.1 0 0 rpy=0 0 0
- added joint joint1: type revolute, parent base_link, child link1, origin xyz=0 0 0 rpy=0 0 0, axis 0 0 1, limit lower=-1.57 upper=1.57 effort=5 velocity=2
- added joint joint2: type revolute, parent link1, child link2, origin xyz=0 0 0.1 rpy=0 0 0, axis 0 1 0, limit lower=-1.57 upper=1.57 effort=5 velocity=2
- added joint joint3: type revolute, parent link2, child link3, origin xyz=0.2 0 0 rpy=0 0 0, axis 0 1 0, limit lower=-1.57 upper=1.57 effort=5 velocity=2
- added joint joint4: type revolute, parent link3, child link4, origin xyz=0.2 0 0 rpy=0 0 0, axis 0 1 0, limit lower=-1.57 upper=1.57 effort=5 velocity=2
- added joint joint5: type revolute, parent link4, child link5, origin xyz=0.16 0 0 rpy=0 0 0, axis 0 0 1, limit lower=-1.57 upper=1.57 effort=5 velocity=2
- added joint joint6: type revolute, parent link5, child link6, origin xyz=0.12 0 0 rpy=0 0 0, axis 0 1 0, limit lower=-1.57 upper=1.57 effort=5 velocity=2

Commit message: Define robot arm model in URDF format
This URDF file describes a robot arm model with multiple links and joints, including a base, segments, and an end effector. Each component has visual, inertial, and collision properties defined.

File: training/robot_arm.urdf (robot description, URDF)
Before this commit: robot placeholder_robot_arm, 1 links, 0 joints
Links:
- added link end_effector, mass 0.1; collision sphere radius=0.02; visual sphere radius=0.02
- added link link_1, mass 0.5; collision box size=0.05 0.05 0.15; visual box size=0.05 0.05 0.15
- added link link_2, mass 0.5; collision box size=0.05 0.05 0.15; visual box size=0.05 0.05 0.15
- added link link_3, mass 0.4; collision box size=0.05 0.05 0.12; visual box size=0.05 0.05 0.12
- added link link_4, mass 0.3; collision box size=0.04 0.04 0.10; visual box size=0.04 0.04 0.10
- added link link_5, mass 0.2; collision box size=0.04 0.04 0.08; visual box size=0.04 0.04 0.08
- link base_link: mass None -> 1.0; geometry collision cylinder length=0.1 radius=0.05; visual cylinder length=0.1 radius=0.05
Joints:
- added joint joint_0: type revolute, parent base_link, child link_1, origin xyz=0 0 0.05 rpy=0 0 0, axis 0 0 1, limit lower=-3.14 upper=3.14 effort=10 velocity=1.0
- added joint joint_1: type revolute, parent link_1, child link_2, origin xyz=0 0 0.15 rpy=0 0 0, axis 0 1 0, limit lower=-1.57 upper=1.57 effort=10 velocity=1.0
- added joint joint_2: type revolute, parent link_2, child link_3, origin xyz=0 0 0.15 rpy=0 0 0, axis 0 1 0, limit lower=-1.57 upper=1.57 effort=10 velocity=1.0
- added joint joint_3: type revolute, parent link_3, child link_4, origin xyz=0 0 0.12 rpy=0 0 0, axis 0 1 0, limit lower=-1.57 upper=1.57 effort=5 velocity=1.0
- added joint joint_4: type revolute, parent link_4, child link_5, origin xyz=0 0 0.10 rpy=0 0 0, axis 0 0 1, limit lower=-3.14 upper=3.14 effort=5 velocity=1.0
- added joint joint_5: type revolute, parent link_5, child end_effector, origin xyz=0 0 0.08 rpy=0 0 0, axis 1 0 0, limit lower=-1.57 upper=1.57 effort=5 velocity=1.0
